File: watch-v4/$watch-v4.sch (KiCad schematic (older format))
At the start: 33 parts, among them J1 CONN_10, P1 array connection, Q1 MOSFET_P, SW1 SPST, SW2 SPST, SW3 SPST, U1 IC_MCP73831, U2 MAX1724, U3 DS3231, U4 LSM9DS0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

Commit message: board errata, new gerber files
Parts:
- added C1: 4.7uf, Capacitors_SMD:C_0402, symbol C-RESCUE-watch-v4
- R3: value R100kΩ -> R10kΩ
Connections:
- net Battery: now also C1.1
- net GND: now also C1.2
- net at C10.1, X1.3: now also U5.38 (XC1); no longer U5.37 (XC2)
- net at 12pf1.2, X1.1: now also U5.37 (XC2); no longer U5.38 (XC1)
Changed lines of the file:
@@
 $EndDescr
 $Comp
-L GND-RESCUE-watch-v4 #PWR17
+L GND-RESCUE-watch-v4 #PWR01
 U 1 1 546D8E5D
 P 9600 600
-F 0 "#PWR17" H 9600 600 30  0001 C CNN
+F 0 "#PWR01" H 9600 600 30  0001 C CNN
 F 1 "GND" H 9600 530 30  0001 C CNN
 F 2 "" H 9600 600 60  0000 C CNN
@@
 $EndComp
 $Comp
-L GND-RESCUE-watch-v4 #PWR13
+L GND-RESCUE-watch-v4 #PWR02
 U 1 1 546D9BFE
 P 8000 2700
-F 0 "#PWR13" H 8000 2700 30  0001 C CNN
+F 0 "#PWR02" H 8000 2700 30  0001 C CNN
 F 1 "GND" H 8000 2630 30  0001 C CNN
 F 2 "" H 8000 2700 60  0000 C CNN
@@
 $EndComp
 $Comp
-L GND-RESCUE-watch-v4 #PWR11
+L GND-RESCUE-watch-v4 #PWR03
 U 1 1 546D9C55
 P 7700 2400
-F 0 "#PWR11" H 7700 2400 30  0001 C CNN
+F 0 "#PWR03" H 7700 2400 30  0001 C CNN
 F 1 "GND" H 7700 2330 30  0001 C CNN
 F 2 "" H 7700 2400 60  0000 C CNN
@@
 $EndComp
 $Comp
-L GND-RESCUE-watch-v4 #PWR10
+L GND-RESCUE-watch-v4 #PWR04
 U 1 1 546D9D6C
 P 7450 2300
-F 0 "#PWR10" H 7450 2300 30  0001 C CNN
+F 0 "#PWR04" H 7450 2300 30  0001 C CNN
 F 1 "GND" H 7450 2230 30  0001 C CNN
 F 2 "" H 7450 2300 60  0000 C CNN
@@
 P 8750 2150
 F 0 "R3" V 8830 2150 40  0000 C CNN
-F 1 "R100kΩ" V 8757 2151 40  0000 C CNN
+F 1 "R10kΩ" V 8757 2151 40  0000 C CNN
 F 2 "Resistors_SMD:R_0402" V 8680 2150 30  0000 C CNN
 F 3 "~" H 8750 2150 30  0000 C CNN
@@
 $EndComp
 $Comp
-L GND-RESCUE-watch-v4 #PWR14
+L GND-RESCUE-watch-v4 #PWR05
 U 1 1 546DA415
 P 8750 2500
-F 0 "#PWR14" H 8750 2500 30  0001 C CNN
+F 0 "#PWR05" H 8750 2500 30  0001 C CNN
 F 1 "GND" H 8750 2430 30  0001 C CNN
 F 2 "" H 8750 2500 60  0000 C CNN
@@
 $EndComp
 $Comp
-L GND-RESCUE-watch-v4 #PWR18
+L GND-RESCUE-watch-v4 #PWR06
 U 1 1 546DAB06
 P 9600 3200
-F 0 "#PWR18" H 9600 3200 30  0001 C CNN
+F 0 "#PWR06" H 9600 3200 30  0001 C CNN
 F 1 "GND" H 9600 3130 30  0001 C CNN
 F 2 "" H 9600 3200 60  0000 C CNN
@@
 VCC
 $Comp
-L GND-RESCUE-watch-v4 #PWR4
+L GND-RESCUE-watch-v4 #PWR07
 U 1 1 546F5D4C
 P 3100 7150
-F 0 "#PWR4" H 3100 7150 30  0001 C CNN
+F 0 "#PWR07" H 3100 7150 30  0001 C CNN
 F 1 "GND" H 3100 7080 30  0001 C CNN
 F 2 "" H 3100 7150 60  0000 C CNN
@@
 $EndComp
 $Comp
-L GND-RESCUE-watch-v4 #PWR12
+L GND-RESCUE-watch-v4 #PWR08
 U 1 1 5470F307
 P 7950 6600
-F 0 "#PWR12" H 7950 6600 30  0001 C CNN
+F 0 "#PWR08" H 7950 6600 30  0001 C CNN
 F 1 "GND" H 7950 6530 30  0001 C CNN
 F 2 "" H 7950 6600 60  0000 C CNN
@@
 $EndComp
 $Comp
-L GND-RESCUE-watch-v4 #PWR16
+L GND-RESCUE-watch-v4 #PWR09
 U 1 1 5470F870
 P 9550 6150
-F 0 "#PWR16" H 9550 6150 30  0001 C CNN
+F 0 "#PWR09" H 9550 6150 30  0001 C CNN
 F 1 "GND" H 9550 6080 30  0001 C CNN
 F 2 "" H 9550 6150 60  0000 C CNN
@@
 VCC
 $Comp
-L GND-RESCUE-watch-v4 #PWR1
+L GND-RESCUE-watch-v4 #PWR010
 U 1 1 54711C87
 P 1250 1550
-F 0 "#PWR1" H 1250 1550 30  0001 C CNN
+F 0 "#PWR010" H 1250 1550 30  0001 C CNN
 F 1 "GND" H 1250 1480 30  0001 C CNN
 F 2 "" H 1250 1550 60  0000 C CNN
@@
 $EndComp
 $Comp
-L GND-RESCUE-watch-v4 #PWR9
+L GND-RESCUE-watch-v4 #PWR011
 U 1 1 5500DCCB
 P 6150 4450
-F 0 "#PWR9" H 6150 4450 30  0001 C CNN
+F 0 "#PWR011" H 6150 4450 30  0001 C CNN
 F 1 "GND" H 6150 4380 30  0001 C CNN
 F 2 "" H 6150 4450 60  0000 C CNN
@@
 $EndComp
 $Comp
-L GND-RESCUE-watch-v4 #PWR5
+L GND-RESCUE-watch-v4 #PWR012
 U 1 1 5501371C
 P 4800 3350
-F 0 "#PWR5" H 4800 3350 30  0001 C CNN
+F 0 "#PWR012" H 4800 3350 30  0001 C CNN
 F 1 "GND" H 4800 3280 30  0001 C CNN
 F 2 "" H 4800 3350 60  0000 C CNN
@@
 $EndComp
 $Comp
-L GND-RESCUE-watch-v4 #PWR3
+L GND-RESCUE-watch-v4 #PWR013
 U 1 1 550137A0
 P 2500 3700
-F 0 "#PWR3" H 2500 3700 30  0001 C CNN
+F 0 "#PWR013" H 2500 3700 30  0001 C CNN
 F 1 "GND" H 2500 3630 30  0001 C CNN
 F 2 "" H 2500 3700 60  0000 C CNN
@@
 $EndComp
 $Comp
-L GND-RESCUE-watch-v4 #PWR6
+L GND-RESCUE-watch-v4 #PWR014
 U 1 1 550A618A
 P 4850 2400
-F 0 "#PWR6" H 4850 2400 30  0001 C CNN
+F 0 "#PWR014" H 4850 2400 30  0001 C CNN
 F 1 "GND" H 4850 2330 30  0001 C CNN
 F 2 "" H 4850 2400 60  0000 C CNN
@@
 $EndComp
 $Comp
-L GND-RESCUE-watch-v4 #PWR2
+L GND-RESCUE-watch-v4 #PWR015
 U 1 1 550BC179
 P 2350 1650
-F 0 "#PWR2" H 2350 1650 30  0001 C CNN
+F 0 "#PWR015" H 2350 1650 30  0001 C CNN
 F 1 "GND" H 2350 1580 30  0001 C CNN
 F 2 "" H 2350 1650 60  0000 C CNN
@@
 $EndComp
 $Comp
-L GND-RESCUE-watch-v4 #PWR15
+L GND-RESCUE-watch-v4 #PWR016
 U 1 1 550BC7D7
 P 9050 4200
-F 0 "#PWR15" H 9050 4200 30  0001 C CNN
+F 0 "#PWR016" H 9050 4200 30  0001 C CNN
 F 1 "GND" H 9050 4130 30  0001 C CNN
 F 2 "" H 9050 4200 60  0000 C CNN
@@
 $EndComp
 $Comp
-L GND-RESCUE-watch-v4 #PWR8
+L GND-RESCUE-watch-v4 #PWR017
 U 1 1 550DE300
 P 5800 2900
-F 0 "#PWR8" H 5800 2900 30  0001 C CNN
+F 0 "#PWR017" H 5800 2900 30  0001 C CNN
 F 1 "GND" H 5800 2830 30  0001 C CNN
 F 2 "" H 5800 2900 60  0000 C CNN
@@
 RX
 $Comp
-L GND-RESCUE-watch-v4 #PWR7
+L GND-RESCUE-watch-v4 #PWR018
 U 1 1 554C655A
 P 4950 850
-F 0 "#PWR7" H 4950 850 30  0001 C CNN
+F 0 "#PWR018" H 4950 850 30  0001 C CNN
 F 1 "GND" H 4950 780 30  0001 C CNN
 F 2 "" H 4950 850 60  0000 C CNN
@@
 	4300 3350 4300 3450
 Wire Wire Line
-	5050 4150 5300 4150
+	4950 4150 5300 4150
 Wire Wire Line
 	5050 4750 5300 4750
@@
 	2400 2700 2650 2700
 Wire Wire Line
-	4800 4150 4800 4600
-Wire Wire Line
-	4600 4000 4800 4150
-Wire Wire Line
-	4650 3900 5050 4150
-Wire Wire Line
-	4300 4000 4600 4000
-Wire Wire Line
-	4300 3900 4650 3900
+	4800 3900 4800 4600
 Text Label 7450 1650 0    60   ~ 0
 Battery
@@
 	1    0    0    -1
 $EndComp
+$Comp
+L C-RESCUE-watch-v4 C1
+U 1 1 55872419
+P 6850 2750
+F 0 "C1" H 6850 2850 40  0000 L CNN
+F 1 "4.7uf" H 6856 2665 40  0000 L CNN
+F 2 "Capacitors_SMD:C_0402" H 6888 2600 30  0000 C CNN
+F 3 "~" H 6850 2750 60  0000 C CNN
+	1    6850 2750
+	1    0    0    -1
+$EndComp
+Text Label 6850 2400 0    60   ~ 0
+Battery
+$Comp
+L GND #PWR019
+U 1 1 558725F3
+P 6850 3200
+F 0 "#PWR019" H 6850 2950 50  0001 C CNN
+F 1 "GND" H 6850 3050 50  0000 C CNN
+F 2 "" H 6850 3200 60  0000 C CNN
+F 3 "" H 6850 3200 60  0000 C CNN
+	1    6850 3200
+	1    0    0    -1
+$EndComp
+Wire Wire Line
+	6850 2400 6850 2550
+Wire Wire Line
+	6850 2950 6850 3200
+Wire Wire Line
+	4950 4150 4950 4000
+Wire Wire Line
+	4950 4000 4300 4000
+Wire Wire Line
+	4800 3900 4300 3900
 $EndSCHEMATC
