File: watch-v4/_saved_watch-v4.sch (KiCad schematic (older format))
At the start: 36 parts, among them J1 CONN_10, P1 array connection, Q1 MOSFET_P, SW1 SPST, SW2 SPST, SW3 SPST, U1 IC_MCP73831, U2 MAX1722, U3 DS3231, U4 LSM9DS0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

Commit message: really should have commited this months ago...
Connections:
- wire segments 139 -> 138
Changed lines of the file:
@@
 	9600 1350 9600 1700
 Wire Wire Line
-	4900 5550 4900 5950
+	4900 5950 4900 5550
 Wire Wire Line
 	5200 4150 5300 4150
@@
 Connection ~ 1400 1150
 Wire Wire Line
-	1400 950  1400 1350
+	1400 1050 1400 1350
 Connection ~ 4900 5950
 Connection ~ 4700 5950
@@
 Wire Wire Line
 	7350 1900 7350 2200
-$Comp
-L GND-RESCUE-watch-v4 #PWR022
-U 1 1 55AF865D
-P 7600 2100
-F 0 "#PWR022" H 7600 2100 30  0001 C CNN
-F 1 "GND" H 7600 2030 30  0001 C CNN
-F 2 "" H 7600 2100 60  0000 C CNN
-F 3 "" H 7600 2100 60  0000 C CNN
-	1    7600 2100
-	0    -1   -1   0
-$EndComp
-Wire Wire Line
-	7350 2100 7600 2100
-Connection ~ 7350 2100
 Wire Wire Line
 	4950 950  4950 1100
