File: watch-v4/_saved_watch-v4.sch (KiCad schematic (older format))
At the start: 38 parts, among them J1 CONN_10, Q1 MOSFET_P, SW1 SPST, SW2 SPST, SW3 SPST, U1 IC_MCP73831, U2 MAX1722, U3 DS3231, U4 LSM9DS0, U5 NRF51822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

Commit message: up to version 5.2
Parts:
- U7: renamed from U?; footprint (none) -> LEDs:Neopixel
Changed lines of the file:
@@
 $EndDescr
 $Comp
-L GND-RESCUE-watch-v4 #PWR01
+L GND-RESCUE-watch-v4 #PWR20
 U 1 1 546D8E5D
 P 9600 1700
-F 0 "#PWR01" H 9600 1700 30  0001 C CNN
+F 0 "#PWR20" H 9600 1700 30  0001 C CNN
 F 1 "GND" H 9600 1630 30  0001 C CNN
 F 2 "" H 9600 1700 60  0000 C CNN
@@
 $EndComp
 $Comp
-L GND-RESCUE-watch-v4 #PWR02
+L GND-RESCUE-watch-v4 #PWR21
 U 1 1 546DAB06
 P 9600 4450
-F 0 "#PWR02" H 9600 4450 30  0001 C CNN
+F 0 "#PWR21" H 9600 4450 30  0001 C CNN
 F 1 "GND" H 9600 4380 30  0001 C CNN
 F 2 "" H 9600 4450 60  0000 C CNN
@@
 VCC
 $Comp
-L GND-RESCUE-watch-v4 #PWR03
+L GND-RESCUE-watch-v4 #PWR4
 U 1 1 546F5D4C
 P 3000 6050
-F 0 "#PWR03" H 3000 6050 30  0001 C CNN
+F 0 "#PWR4" H 3000 6050 30  0001 C CNN
 F 1 "GND" H 3000 5980 30  0001 C CNN
 F 2 "" H 3000 6050 60  0000 C CNN
@@
 $EndComp
 $Comp
-L GND-RESCUE-watch-v4 #PWR04
+L GND-RESCUE-watch-v4 #PWR6
 U 1 1 5470F307
 P 4650 7900
-F 0 "#PWR04" H 4650 7900 30  0001 C CNN
+F 0 "#PWR6" H 4650 7900 30  0001 C CNN
 F 1 "GND" H 4650 7830 30  0001 C CNN
 F 2 "" H 4650 7900 60  0000 C CNN
@@
 $EndComp
 $Comp
-L GND-RESCUE-watch-v4 #PWR05
+L GND-RESCUE-watch-v4 #PWR13
 U 1 1 5470F870
 P 6250 7450
-F 0 "#PWR05" H 6250 7450 30  0001 C CNN
+F 0 "#PWR13" H 6250 7450 30  0001 C CNN
 F 1 "GND" H 6250 7380 30  0001 C CNN
 F 2 "" H 6250 7450 60  0000 C CNN
@@
 VCC
 $Comp
-L GND-RESCUE-watch-v4 #PWR06
+L GND-RESCUE-watch-v4 #PWR1
 U 1 1 54711C87
 P 1250 1550
-F 0 "#PWR06" H 1250 1550 30  0001 C CNN
+F 0 "#PWR1" H 1250 1550 30  0001 C CNN
 F 1 "GND" H 1250 1480 30  0001 C CNN
 F 2 "" H 1250 1550 60  0000 C CNN
@@
 $EndComp
 $Comp
-L GND-RESCUE-watch-v4 #PWR07
+L GND-RESCUE-watch-v4 #PWR11
 U 1 1 5500DCCB
 P 6150 4450
-F 0 "#PWR07" H 6150 4450 30  0001 C CNN
+F 0 "#PWR11" H 6150 4450 30  0001 C CNN
 F 1 "GND" H 6150 4380 30  0001 C CNN
 F 2 "" H 6150 4450 60  0000 C CNN
@@
 $EndComp
 $Comp
-L GND-RESCUE-watch-v4 #PWR08
+L GND-RESCUE-watch-v4 #PWR7
 U 1 1 5501371C
 P 4800 3350
-F 0 "#PWR08" H 4800 3350 30  0001 C CNN
+F 0 "#PWR7" H 4800 3350 30  0001 C CNN
 F 1 "GND" H 4800 3280 30  0001 C CNN
 F 2 "" H 4800 3350 60  0000 C CNN
@@
 $EndComp
 $Comp
-L GND-RESCUE-watch-v4 #PWR09
+L GND-RESCUE-watch-v4 #PWR3
 U 1 1 550137A0
 P 2500 3700
-F 0 "#PWR09" H 2500 3700 30  0001 C CNN
+F 0 "#PWR3" H 2500 3700 30  0001 C CNN
 F 1 "GND" H 2500 3630 30  0001 C CNN
 F 2 "" H 2500 3700 60  0000 C CNN
@@
 $EndComp
 $Comp
-L GND-RESCUE-watch-v4 #PWR010
+L GND-RESCUE-watch-v4 #PWR2
 U 1 1 550BC179
 P 2350 1650
-F 0 "#PWR010" H 2350 1650 30  0001 C CNN
+F 0 "#PWR2" H 2350 1650 30  0001 C CNN
 F 1 "GND" H 2350 1580 30  0001 C CNN
 F 2 "" H 2350 1650 60  0000 C CNN
@@
 $EndComp
 $Comp
-L GND-RESCUE-watch-v4 #PWR011
+L GND-RESCUE-watch-v4 #PWR10
 U 1 1 550BC7D7
 P 5750 5500
-F 0 "#PWR011" H 5750 5500 30  0001 C CNN
+F 0 "#PWR10" H 5750 5500 30  0001 C CNN
 F 1 "GND" H 5750 5430 30  0001 C CNN
 F 2 "" H 5750 5500 60  0000 C CNN
@@
 Regulator_In
 $Comp
-L GND #PWR012
+L GND #PWR15
 U 1 1 55AF0371
 P 7350 1400
-F 0 "#PWR012" H 7350 1150 50  0001 C CNN
+F 0 "#PWR15" H 7350 1150 50  0001 C CNN
 F 1 "GND" H 7350 1250 50  0000 C CNN
 F 2 "" H 7350 1400 60  0000 C CNN
@@
 $EndComp
 $Comp
-L GND #PWR013
+L GND #PWR22
 U 1 1 55AF081A
 P 10000 2100
-F 0 "#PWR013" H 10000 1850 50  0001 C CNN
+F 0 "#PWR22" H 10000 1850 50  0001 C CNN
 F 1 "GND" H 10000 1950 50  0000 C CNN
 F 2 "" H 10000 2100 60  0000 C CNN
@@
 $EndComp
 $Comp
-L GND #PWR014
+L GND #PWR14
 U 1 1 55AF0E1B
 P 6950 2200
-F 0 "#PWR014" H 6950 1950 50  0001 C CNN
+F 0 "#PWR14" H 6950 1950 50  0001 C CNN
 F 1 "GND" H 6950 2050 50  0000 C CNN
 F 2 "" H 6950 2200 60  0000 C CNN
@@
 $EndComp
 $Comp
-L GND #PWR015
+L GND #PWR12
 U 1 1 55AF193D
 P 6250 1500
-F 0 "#PWR015" H 6250 1250 50  0001 C CNN
+F 0 "#PWR12" H 6250 1250 50  0001 C CNN
 F 1 "GND" H 6250 1350 50  0000 C CNN
 F 2 "" H 6250 1500 60  0000 C CNN
@@
 VBAT
 $Comp
-L GND #PWR016
+L GND #PWR18
 U 1 1 55AF2A49
 P 7900 3000
-F 0 "#PWR016" H 7900 2750 50  0001 C CNN
+F 0 "#PWR18" H 7900 2750 50  0001 C CNN
 F 1 "GND" H 7900 2850 50  0000 C CNN
 F 2 "" H 7900 3000 60  0000 C CNN
@@
 Connection ~ 8050 3350
 $Comp
-L GND #PWR017
+L GND #PWR19
 U 1 1 55AF413B
 P 8050 3800
-F 0 "#PWR017" H 8050 3550 50  0001 C CNN
+F 0 "#PWR19" H 8050 3550 50  0001 C CNN
 F 1 "GND" H 8050 3650 50  0000 C CNN
 F 2 "" H 8050 3800 60  0000 C CNN
@@
 $EndComp
 $Comp
-L GND #PWR018
+L GND #PWR16
 U 1 1 55AF64EA
 P 7350 2200
-F 0 "#PWR018" H 7350 1950 50  0001 C CNN
+F 0 "#PWR16" H 7350 1950 50  0001 C CNN
 F 1 "GND" H 7350 2050 50  0000 C CNN
 F 2 "" H 7350 2200 60  0000 C CNN
@@
 	7350 1900 7350 2200
 $Comp
-L GND-RESCUE-watch-v4 #PWR019
+L GND-RESCUE-watch-v4 #PWR17
 U 1 1 55AF865D
 P 7600 2100
-F 0 "#PWR019" H 7600 2100 30  0001 C CNN
+F 0 "#PWR17" H 7600 2100 30  0001 C CNN
 F 1 "GND" H 7600 2030 30  0001 C CNN
 F 2 "" H 7600 2100 60  0000 C CNN
@@
 	1400 1050 1400 1350
 $Comp
-L GND #PWR020
+L GND #PWR9
 U 1 1 56272AEE
 P 5450 3500
-F 0 "#PWR020" H 5450 3250 50  0001 C CNN
+F 0 "#PWR9" H 5450 3250 50  0001 C CNN
 F 1 "GND" H 5450 3350 50  0000 C CNN
 F 2 "" H 5450 3500 60  0000 C CNN
@@
 $EndComp
 $Comp
-L GND #PWR021
+L GND #PWR8
 U 1 1 56272B62
 P 5450 2800
-F 0 "#PWR021" H 5450 2550 50  0001 C CNN
+F 0 "#PWR8" H 5450 2550 50  0001 C CNN
 F 1 "GND" H 5450 2650 50  0000 C CNN
 F 2 "" H 5450 2800 60  0000 C CNN
@@
 SW3
 $Comp
-L GND #PWR022
+L GND #PWR23
 U 1 1 570216B0
 P 10300 5500
-F 0 "#PWR022" H 10300 5250 50  0001 C CNN
+F 0 "#PWR23" H 10300 5250 50  0001 C CNN
 F 1 "GND" H 10300 5350 50  0000 C CNN
 F 2 "" H 10300 5500 60  0000 C CNN
@@
 	5600 3550 5800 3550
 $Comp
-L GND #PWR023
+L GND #PWR5
 U 1 1 570C1180
 P 4170 850
-F 0 "#PWR023" H 4170 600 50  0001 C CNN
+F 0 "#PWR5" H 4170 600 50  0001 C CNN
 F 1 "GND" H 4170 700 50  0000 C CNN
 F 2 "" H 4170 850 60  0000 C CNN
@@
 Backlight
 $Comp
-L NeoPixel U?
+L NeoPixel U7
 U 1 1 570D0584
 P 4850 1050
-F 0 "U?" H 4550 1390 50  0000 C CNN
+F 0 "U7" H 4550 1390 50  0000 C CNN
 F 1 "NeoPixel" H 4650 700 50  0000 C CNN
-F 2 "" H 4775 1000 50  0000 C CNN
+F 2 "LEDs:Neopixel" H 4775 1000 50  0000 C CNN
 F 3 "" H 4775 1000 50  0000 C CNN
 	1    4850 1050
