File: watch-v4/_saved_watch-v4.sch (KiCad schematic (older format))
At the start: 44 parts, among them J1 CONN_10, P1 Expansion Header, Q1 MOSFET_P, Q2 BSS138, U1 IC_MCP73831, U2 MAX1722, U3 DS3231, U4 LSM9DS0, U5 NRF51822, U6 BALUN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

Commit message: further traces routed, still more work to go
Connections:
- net SCL: now also P1.3 (P3); no longer P1.4 (P4)
- net SDA: now also P1.4 (P4); no longer P1.3 (P3)
Changed lines of the file:
@@
 Text Label 3175 8200 0    60   ~ 0
 SCL
+Text Label 1250 4850 2    60   ~ 0
+SDA
 Text Label 1250 4750 2    60   ~ 0
-SDA
-Text Label 1250 4850 2    60   ~ 0
 SCL
 Text Label 14975 5450 2    60   ~ 0
