File: watch-v4/watch-v4.sch (KiCad schematic (older format))
At the start: 36 parts, among them J1 CONN_10, P1 array connection, Q1 MOSFET_P, SW1 SPST, SW2 SPST, SW3 SPST, U1 IC_MCP73831, U2 MAX1722, U3 DS3231, U4 LSM9DS0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

Commit message: add 4.5 gerbers
Parts:
- removed C12: 2.2nf, Capacitors_SMD:C_0603, symbol CAPACITOR_NPOL-0402
- U6: footprint watch-v4:BALUN -> watch-v4:BALUN-6
Connections:
- net DISPLAY_SCK: now also J1.3 (P3); no longer J1.1 (P1)
- net DISPLAY_SS: now also J1.1 (P1); no longer J1.3 (P3)
- net GND: now also U6.2 (GND), U6.5 (GND); no longer U6.4 (ANT_OUT)
- net VCC: no longer J1.4 (P4)
- net at U5.30 (VDD_PA): no longer U6.3 (ANT_OUT)
- net at U5.31 (ANT1): now also U5.32 (ANT2), U6.1 (ANT_IN); no longer U6.2 (GND)
- net at ANT1.1: now also U6.3 (ANT_OUT), U6.4 (ANT_OUT); no longer U6.5 (GND)
Other:
- moved on the sheet: U6
Changed lines of the file:
@@
 Text GLabel 1950 3500 0    60   Input ~ 0
 DISPLAY_SS
+Text GLabel 1200 600  0    60   Input ~ 0
+DISPLAY_SS
 Text GLabel 1200 900  0    60   Input ~ 0
-DISPLAY_SS
-Text GLabel 1200 600  0    60   Input ~ 0
 DISPLAY_SCK
 Text GLabel 1200 750  0    60   Input ~ 0
@@
 L BALUN U6
 U 1 1 550A5E51
-P 5300 3000
-F 0 "U6" H 5300 3250 60  0000 C CNN
-F 1 "BALUN" H 5300 3350 60  0000 C CNN
-F 2 "watch-v4:BALUN" H 5300 3150 60  0001 C CNN
-F 3 "" H 5300 3150 60  0000 C CNN
-	1    5300 3000
-	1    0    0    -1
-$EndComp
-$Comp
-L CAPACITOR_NPOL-0402 C12
-U 1 1 550A5FE9
-P 4850 2700
-F 0 "C12" V 5050 2550 50  0000 L BNN
-F 1 "2.2nf" V 4950 2500 50  0000 L BNN
-F 2 "Capacitors_SMD:C_0603" H 4850 2850 50  0001 C CNN
-F 3 "" H 4850 2700 60  0000 C CNN
-	1    4850 2700
-	-1   0    0    1
-$EndComp
-$Comp
-L GND-RESCUE-watch-v4 #PWR010
-U 1 1 550A618A
-P 4850 2400
-F 0 "#PWR010" H 4850 2400 30  0001 C CNN
-F 1 "GND" H 4850 2330 30  0001 C CNN
-F 2 "" H 4850 2400 60  0000 C CNN
-F 3 "" H 4850 2400 60  0000 C CNN
-	1    4850 2400
-	-1   0    0    1
+P 5400 3150
+F 0 "U6" H 5400 3400 60  0000 C CNN
+F 1 "BALUN" H 5400 3500 60  0000 C CNN
+F 2 "watch-v4:BALUN-6" H 5400 3300 60  0001 C CNN
+F 3 "" H 5400 3300 60  0000 C CNN
+	1    5400 3150
+	0    1    1    0
 $EndComp
 $Comp
@@
 $EndComp
 $Comp
-L GND-RESCUE-watch-v4 #PWR011
+L GND-RESCUE-watch-v4 #PWR010
 U 1 1 550BC179
 P 2350 1650
-F 0 "#PWR011" H 2350 1650 30  0001 C CNN
+F 0 "#PWR010" H 2350 1650 30  0001 C CNN
 F 1 "GND" H 2350 1580 30  0001 C CNN
 F 2 "" H 2350 1650 60  0000 C CNN
@@
 $EndComp
 $Comp
-L GND-RESCUE-watch-v4 #PWR012
+L GND-RESCUE-watch-v4 #PWR011
 U 1 1 550BC7D7
 P 5750 5500
-F 0 "#PWR012" H 5750 5500 30  0001 C CNN
+F 0 "#PWR011" H 5750 5500 30  0001 C CNN
 F 1 "GND" H 5750 5430 30  0001 C CNN
 F 2 "" H 5750 5500 60  0000 C CNN
@@
 	1    4600 3550
 	1    0    0    -1
-$EndComp
-$Comp
-L GND-RESCUE-watch-v4 #PWR013
-U 1 1 550DE300
-P 5800 2900
-F 0 "#PWR013" H 5800 2900 30  0001 C CNN
-F 1 "GND" H 5800 2830 30  0001 C CNN
-F 2 "" H 5800 2900 60  0000 C CNN
-F 3 "" H 5800 2900 60  0000 C CNN
-	1    5800 2900
-	0    -1   -1   0
 $EndComp
 $Comp
@@
 RX
 $Comp
-L GND-RESCUE-watch-v4 #PWR014
+L GND-RESCUE-watch-v4 #PWR012
 U 1 1 554C655A
 P 5050 850
-F 0 "#PWR014" H 5050 850 30  0001 C CNN
+F 0 "#PWR012" H 5050 850 30  0001 C CNN
 F 1 "GND" H 5050 780 30  0001 C CNN
 F 2 "" H 5050 850 60  0000 C CNN
@@
 EXTVCC
 $Comp
-L GND #PWR015
+L GND #PWR013
 U 1 1 55AF0371
 P 7350 1400
-F 0 "#PWR015" H 7350 1150 50  0001 C CNN
+F 0 "#PWR013" H 7350 1150 50  0001 C CNN
 F 1 "GND" H 7350 1250 50  0000 C CNN
 F 2 "" H 7350 1400 60  0000 C CNN
@@
 $EndComp
 $Comp
-L GND #PWR016
+L GND #PWR014
 U 1 1 55AF081A
 P 10000 2100
-F 0 "#PWR016" H 10000 1850 50  0001 C CNN
+F 0 "#PWR014" H 10000 1850 50  0001 C CNN
 F 1 "GND" H 10000 1950 50  0000 C CNN
 F 2 "" H 10000 2100 60  0000 C CNN
@@
 $EndComp
 $Comp
-L GND #PWR017
+L GND #PWR015
 U 1 1 55AF0E1B
 P 6950 2200
-F 0 "#PWR017" H 6950 1950 50  0001 C CNN
+F 0 "#PWR015" H 6950 1950 50  0001 C CNN
 F 1 "GND" H 6950 2050 50  0000 C CNN
 F 2 "" H 6950 2200 60  0000 C CNN
@@
 $EndComp
 $Comp
-L GND #PWR018
+L GND #PWR016
 U 1 1 55AF193D
 P 6250 1500
-F 0 "#PWR018" H 6250 1250 50  0001 C CNN
+F 0 "#PWR016" H 6250 1250 50  0001 C CNN
 F 1 "GND" H 6250 1350 50  0000 C CNN
 F 2 "" H 6250 1500 60  0000 C CNN
@@
 VBAT
 $Comp
-L GND #PWR019
+L GND #PWR017
 U 1 1 55AF2A49
 P 7900 3000
-F 0 "#PWR019" H 7900 2750 50  0001 C CNN
+F 0 "#PWR017" H 7900 2750 50  0001 C CNN
 F 1 "GND" H 7900 2850 50  0000 C CNN
 F 2 "" H 7900 3000 60  0000 C CNN
@@
 	9600 1350 9600 1700
 Wire Wire Line
-	4900 5550 4900 5950
+	4900 5950 4900 5550
 Wire Wire Line
 	5200 4150 5300 4150
@@
 Wire Wire Line
 	5050 850  5050 1100
-Wire Wire Line
-	5650 2900 5800 2900
 Connection ~ 4600 3350
 Wire Wire Line
@@
 	900  3950 1000 3950
 Wire Wire Line
-	4850 2600 4850 2400
-Wire Wire Line
-	4850 2900 4950 2900
-Wire Wire Line
-	4850 2950 4850 2900
-Wire Wire Line
-	4300 2950 4850 2950
-Wire Wire Line
-	5650 3050 5850 3050
-Wire Wire Line
-	4300 3200 4950 3200
+	4950 3200 4300 3200
 Wire Wire Line
 	4900 3100 4950 3050
@@
 Connection ~ 1400 1250
 Connection ~ 1400 1150
-Wire Wire Line
-	1400 950  1400 1350
 Connection ~ 4900 5950
 Connection ~ 4700 5950
@@
 Connection ~ 8050 3350
 $Comp
-L GND #PWR020
+L GND #PWR018
 U 1 1 55AF413B
 P 8050 3800
-F 0 "#PWR020" H 8050 3550 50  0001 C CNN
+F 0 "#PWR018" H 8050 3550 50  0001 C CNN
 F 1 "GND" H 8050 3650 50  0000 C CNN
 F 2 "" H 8050 3800 60  0000 C CNN
@@
 $EndComp
 $Comp
-L GND #PWR021
+L GND #PWR019
 U 1 1 55AF64EA
 P 7350 2200
-F 0 "#PWR021" H 7350 1950 50  0001 C CNN
+F 0 "#PWR019" H 7350 1950 50  0001 C CNN
 F 1 "GND" H 7350 2050 50  0000 C CNN
 F 2 "" H 7350 2200 60  0000 C CNN
@@
 	7350 1900 7350 2200
 $Comp
-L GND-RESCUE-watch-v4 #PWR022
+L GND-RESCUE-watch-v4 #PWR020
 U 1 1 55AF865D
 P 7600 2100
-F 0 "#PWR022" H 7600 2100 30  0001 C CNN
+F 0 "#PWR020" H 7600 2100 30  0001 C CNN
 F 1 "GND" H 7600 2030 30  0001 C CNN
 F 2 "" H 7600 2100 60  0000 C CNN
@@
 Wire Wire Line
 	4950 950  4950 1100
+Wire Wire Line
+	1400 1050 1400 1350
+Wire Wire Line
+	5500 2800 5850 2800
+Wire Wire Line
+	5850 2800 5850 3500
+Wire Wire Line
+	5850 3500 5500 3500
+Connection ~ 5850 3050
+Wire Wire Line
+	4950 2800 4950 3200
+Wire Wire Line
+	4950 2800 5200 2800
+Connection ~ 4950 3050
+$Comp
+L GND #PWR021
+U 1 1 56272AEE
+P 5350 3550
+F 0 "#PWR021" H 5350 3300 50  0001 C CNN
+F 1 "GND" H 5350 3400 50  0000 C CNN
+F 2 "" H 5350 3550 60  0000 C CNN
+F 3 "" H 5350 3550 60  0000 C CNN
+	1    5350 3550
+	1    0    0    -1
+$EndComp
+$Comp
+L GND #PWR022
+U 1 1 56272B62
+P 5350 2700
+F 0 "#PWR022" H 5350 2450 50  0001 C CNN
+F 1 "GND" H 5350 2550 50  0000 C CNN
+F 2 "" H 5350 2700 60  0000 C CNN
+F 3 "" H 5350 2700 60  0000 C CNN
+	1    5350 2700
+	-1   0    0    1
+$EndComp
+Wire Wire Line
+	5350 2700 5350 2800
+Wire Wire Line
+	5350 3550 5350 3500
 $EndSCHEMATC
