File: watch-v4/watch-v4.sch (KiCad schematic (older format))
At the start: 38 parts, among them J1 CONN_10, Q1 MOSFET_P, SW1 SPST, SW2 SPST, SW3 SPST, U1 IC_MCP73831, U2 MAX1722, U3 DS3231, U4 LSM9DS0, U5 NRF51822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

Commit message: save v5.2
Parts:
- U7: renamed from U?; footprint (none) -> LEDs:Neopixel
Connections:
- net labels added: Accel_INT, ClockINT
Changed lines of the file:
@@
 	5600 6950 5800 6950
-Wire Wire Line
-	4100 6250 4200 6250
-Wire Wire Line
-	4100 6850 4100 6250
 Wire Wire Line
 	4200 6850 4100 6850
@@
 Backlight
 $Comp
-L NeoPixel U?
+L NeoPixel U7
 U 1 1 570D0584
 P 4850 1050
-F 0 "U?" H 4550 1390 50  0000 C CNN
+F 0 "U7" H 4550 1390 50  0000 C CNN
 F 1 "NeoPixel" H 4650 700 50  0000 C CNN
-F 2 "" H 4775 1000 50  0000 C CNN
+F 2 "LEDs:Neopixel" H 4775 1000 50  0000 C CNN
 F 3 "" H 4775 1000 50  0000 C CNN
 	1    4850 1050
@@
 Wire Wire Line
 	5300 850  5550 850
+Text Label 4300 5000 0    60   ~ 0
+ClockINT
+Text Label 4300 5100 0    60   ~ 0
+Accel_INT
+Text Label 3350 6950 0    60   ~ 0
+Accel_INT
+Text GLabel 4100 6850 0    60   Input ~ 0
+VCC
+Wire Wire Line
+	3350 6950 4200 6950
+Text Label 750  6350 0    60   ~ 0
+ClockINT
+Wire Wire Line
+	750  6350 1350 6350
 $EndSCHEMATC

Commit message: save schematic changes for 5.4
Parts:
- removed R4, R7, R8: 10kΩ, Resistors_SMD:R_0603, symbol R-RESCUE-watch-v4
- removed SW1, SW2, SW3: SPST, watch-v4:SW_Tactile_SPST_Angled_no_anchors, symbol SPST
Connections:
- wire segments 147 -> 133
Other:
- moved on the sheet: 12pf1, ANT1, C1, C10, C13, C14, C2, C3, C5, C6, C7, C8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

Commit message: v6 schematic updates
* add expansion header
* remove buttons
* fix radio decoupling, gnd connections
* change backlight to mosfet/standard leds
* add battery connection through voltage divider
* clock INT pullup on schematic now
Parts:
- removed U7: NeoPixel, LEDs:Neopixel, symbol NeoPixel
- added C11: 2n2, symbol C_Small
- added C12: 1u, symbol C_Small
- added C4: 100n, symbol C_Small
- added C9: 47n, symbol C_Small
- added D3, D4, D5: LED, LEDs:LED-0603, symbol LED
- added P1: Expansion Header, symbol CONN_01X12
- added Q2: BSS138, SOT-23, symbol BSS138
- added R4: 10k, symbol R_Small
- added R7, R8: 10M, symbol R_Small
- added R9: 47, symbol R_Small
- C14: value 0.1uf -> 1nf
Connections:
- net Backlight: now also Q2.1 (G)
- net ClockINT: now also R4.2
- net GND: now also C11.2, C12.2, C4.2, C9.2, P1.2 (P2), Q2.2 (S), R8.2; no longer U6.2 (GND)
- net SCL: now also P1.4 (P4)
- net SDA: now also P1.3 (P3)
- net VBAT: now also R7.1
- net VCC: now also P1.1 (P1), R4.1, R9.1
- net EX11: now reaches U5.17 (P0.11)
- net EX11: now also P1.8 (P8)
- net EX12: now reaches U5.18 (P0.12)
- net EX12: now also P1.9 (P9)
- net EX13: now reaches U5.19 (P0.13)
- net EX13: now also P1.10 (P10)
- net EX14: now reaches U5.20 (P0.14)
- net EX14: now also P1.11 (P11)
- net EX15: now reaches U5.21 (P0.15)
- net EX15: now also P1.12 (P12)
- net BatterySense: now reaches U5.22 (P0.16)
- net BatterySense: now also C12.1, R7.2, R8.1
- net at U5.29 (DEC2): now also C9.1
- net VDD_PA: now reaches U5.30 (VDD_PA)
- net VDD_PA: now also U6.2 (GND), C11.1
- net Bal1: now reaches U5.31 (ANT1)
- net Bal1: now also U6.3 (balanced_1); no longer U6.4 (bal_2)
- net Bal2: now reaches U5.32 (ANT2)
- net Bal2: now also U6.4 (bal_2); no longer U6.3 (balanced_1)
- net at U5.39 (DEC1): now also C4.1
- net SW1 renamed EX8
- net EX8: now also P1.5 (P5)
- net SW2 renamed EX9
- net EX9: now also P1.6 (P6)
- net SW3 renamed EX10
- net EX10: now also P1.7 (P7)
- new net: D3.1 (K), D4.1 (K), D5.1 (K), Q2.3 (D)
- new net: D3.2 (A), D4.2 (A), D5.2 (A), R9.2
Other:
- moved on the sheet: ANT1, J1, U6

Commit message: cleanup
Changed lines of the file:
@@
 	12825 3825 13025 3825
 Wire Wire Line
-	12625 2975 12625 3525
+	12625 2975 12625 3325
+Wire Wire Line
+	12625 3325 12625 3525
 Wire Wire Line
 	12125 3825 12425 3825
@@
 Connection ~ 4725 2425
 Wire Wire Line
-	4425 2425 4925 2425
+	4425 2425 4725 2425
+Wire Wire Line
+	4725 2425 4925 2425
 Wire Wire Line
 	4725 2825 4925 2825
@@
 	6200 7950 6200 7550
 Wire Wire Line
-	5750 7950 6200 7950
+	5750 7950 6000 7950
+Wire Wire Line
+	6000 7950 6200 7950
 Connection ~ 2475 1375
 Wire Wire Line
@@
 Wire Wire Line
 	2475 725  2475 825
-Wire Wire Line
-	2275 3225 2775 3225
 Wire Wire Line
 	4925 3675 5175 3825
@@
 Connection ~ 5725 3525
 Wire Wire Line
-	5725 3225 5725 3825
-Wire Wire Line
-	5625 3525 6275 3525
-Wire Wire Line
-	5175 3825 5425 3825
+	5725 3225 5725 3525
+Wire Wire Line
+	5725 3525 5725 3825
+Wire Wire Line
+	5625 3525 5725 3525
+Wire Wire Line
+	5725 3525 6275 3525
+Wire Wire Line
+	5175 3825 5325 3825
+Wire Wire Line
+	5325 3825 5425 3825
 Wire Wire Line
 	4425 2425 4425 2525
@@
 	2775 1375 2775 1425
 Wire Wire Line
-	2275 1375 2775 1375
+	2275 1375 2475 1375
+Wire Wire Line
+	2475 1375 2775 1375
 Wire Wire Line
 	2775 2775 2625 2775
@@
 Connection ~ 5900 8350
 Wire Wire Line
-	5300 8350 6200 8350
+	5300 8350 5800 8350
+Wire Wire Line
+	5800 8350 5900 8350
+Wire Wire Line
+	5900 8350 6000 8350
+Wire Wire Line
+	6000 8350 6200 8350
 Connection ~ 6000 7950
 Wire Wire Line
@@
 Connection ~ 5850 10150
 Wire Wire Line
-	5750 10150 6250 10150
+	5750 10150 5850 10150
+Wire Wire Line
+	5850 10150 6050 10150
+Wire Wire Line
+	6050 10150 6150 10150
+Wire Wire Line
+	6150 10150 6250 10150
 Connection ~ 1275 10100
 Wire Wire Line
@@
 	3225 8900 2875 8900
 Wire Wire Line
-	1025 8900 1425 8900
+	1025 8900 1225 8900
+Wire Wire Line
+	1225 8900 1425 8900
 Wire Wire Line
 	2875 8750 3075 8750
@@
 	15375 3475 15575 3475
 Wire Wire Line
-	14575 3475 14575 4025
+	14575 3475 14575 3925
+Wire Wire Line
+	14575 3925 14575 4025
 Wire Wire Line
 	14775 3475 14575 3475
@@
 Regulator_In
 Wire Wire Line
-	13025 3325 13675 3325
+	13025 3325 13525 3325
+Wire Wire Line
+	13525 3325 13675 3325
 $Comp
 L C C1
@@
 $EndComp
 Wire Wire Line
-	12825 1875 12825 2175
+	12825 1875 12825 2075
+Wire Wire Line
+	12825 2075 12825 2175
 $Comp
 L GND-RESCUE-watch-v4 #PWR19
@@
 Connection ~ 12825 2075
 Wire Wire Line
-	10750 5225 10750 5525
+	10750 5225 10750 5325
+Wire Wire Line
+	10750 5325 10750 5425
+Wire Wire Line
+	10750 5425 10750 5525
 $Comp
 L GND #PWR7
@@
 	0    -1   -1   0
 $EndComp
-Text Label 2275 2975 0    60   ~ 0
+Text Label 2775 3025 2    60   ~ 0
 EX8
-Wire Wire Line
-	2275 2975 2775 2975
-Wire Wire Line
-	2775 2975 2775 3025
-Text Label 2275 3125 0    60   ~ 0
+Text Label 2775 3125 2    60   ~ 0
 EX9
-Wire Wire Line
-	2275 3125 2775 3125
-Text Label 2275 3225 0    60   ~ 0
+Text Label 2775 3225 2    60   ~ 0
 EX10
 Wire Wire Line
@@
 Wire Wire Line
 	10720 6825 10925 6825
-Text Label 2275 3425 0    60   ~ 0
+Text Label 2775 3425 2    60   ~ 0
 EX12
-Text Label 2275 3325 0    60   ~ 0
+Text Label 2775 3325 2    60   ~ 0
 EX11
-Text Label 2275 3525 0    60   ~ 0
+Text Label 2775 3525 2    60   ~ 0
 EX13
-Text Label 2275 3625 0    60   ~ 0
+Text Label 2775 3625 2    60   ~ 0
 EX14
-Text Label 2275 3725 0    60   ~ 0
+Text Label 2775 3725 2    60   ~ 0
 EX15
-Wire Wire Line
-	2275 3325 2775 3325
-Wire Wire Line
-	2275 3425 2775 3425
-Wire Wire Line
-	2275 3525 2775 3525
-Wire Wire Line
-	2275 3625 2775 3625
-Wire Wire Line
-	2275 3725 2775 3725
 Wire Wire Line
 	10425 7225 10925 7225
@@
 	11025 2350 10775 2350
 Wire Wire Line
-	11025 2550 11025 2800
+	11025 2550 11025 2675
+Wire Wire Line
+	11025 2675 11025 2800
 $Comp
 L GND #PWR13
@@
 	11025 3025 11375 3025
 Wire Wire Line
-	11025 3000 11025 3100
+	11025 3000 11025 3025
+Wire Wire Line
+	11025 3025 11025 3100
 Connection ~ 11025 3025
 $Comp
@@
 	1425 9100 1425 9050
 Wire Wire Line
-	975  9100 1425 9100
+	975  9100 1225 9100
+Wire Wire Line
+	1225 9100 1425 9100
 Connection ~ 1225 9100
 $Comp
@@
 	8325 4525 8500 4525
 Wire Wire Line
-	8500 4525 8500 5175
+	8500 4525 8500 4850
+Wire Wire Line
+	8500 4850 8500 5175
 Connection ~ 8500 4850
 Wire Wire Line
-	8900 4525 8900 5375
+	8900 4525 8900 4850
+Wire Wire Line
+	8900 4850 8900 5175
+Wire Wire Line
+	8900 5175 8900 5375
 Connection ~ 8900 4850
 Connection ~ 8900 5175

Commit message: get rid of the global labels, tidy things up a bit
Connections:
- net SCL: now also R5.1, U3.7 (SDA); no longer R6.1, U3.8 (SCL)
- net SDA: now also R6.1, U3.8 (SCL); no longer R5.1, U3.7 (SDA)
- net DISPLAY_MOSI renamed Display_MOSI
- net DISPLAY_SCK renamed Display_SCK
- net DISPLAY_SS renamed Display_SS
Other:
- moved on the sheet: 12pf1, ANT1, C10, C11, C13, C14, C4, C9, U5, U6, X1

Commit message: more cleanup
Connections:
- net XC2: now reaches 12pf1.2, U5.37 (XC2), X1.1
- net XC1: now reaches C10.1, U5.38 (XC1), X1.3
Other:
- note added: "I2C"
- note added: "MCU/Radio"
- note added: "Power/Charging"
- moved on the sheet: 12pf1, C10, C5, C6, C7, C8, D3, D4, D5, J1, P1, Q2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

Commit message: further v6 work; incomplete
Parts:
- C11, C12, C4, C9: footprint (none) -> Capacitors_SMD:C_0603
- D2, D3, D4, D5: footprint LEDs:LED-0603 -> Capacitors_SMD:C_0603
- LIPOLY1: footprint watch-v4:Pin_Header_Straight_1x02 -> Socket_Strips:molex_2_pos
- P1: footprint (none) -> Socket_Strips:Socket_Strip_Straight_1x12_small
- Q2: footprint SOT-23 -> TO_SOT_Packages_SMD:SOT-23
- R4, R7, R8, R9: footprint (none) -> Resistors_SMD:R_0603
Connections:
- net Bal1: now also U6.4 (bal_2); no longer U6.3 (balanced_1)
- net Bal2: now also U6.3 (balanced_1); no longer U6.4 (bal_2)
- net GND: now also U6.2 (GND); no longer U6.5 (GND)
- net VDD_PA: now also U6.5 (GND); no longer U6.2 (GND)
Other:
- moved on the sheet: C11, D3, D4, D5, P1, Q2, R9

Commit message: top layer components mostly routed
Connections:
- net GND: now also P1.1 (P1); no longer P1.2 (P2)
- net RX: now also XL1.3 (D+); no longer XL1.2 (D-)
- net SCL: now also P1.3 (P3); no longer P1.4 (P4)
- net SDA: now also P1.4 (P4); no longer P1.3 (P3)
- net TX: now also XL1.2 (D-); no longer XL1.3 (D+)
- net VCC: now also P1.2 (P2); no longer P1.1 (P1)
Changed lines of the file:
@@
 Text Label 15175 1625 1    60   ~ 0
 Reset
+Text Label 15375 1625 1    60   ~ 0
+TX
 Text Label 15275 1625 1    60   ~ 0
-TX
-Text Label 15375 1625 1    60   ~ 0
 RX
 Text Label 2400 4850 0    60   ~ 0
@@
 L GND-RESCUE-watch-v4 #PWR023
 U 1 1 58005D02
-P 850 4650
-F 0 "#PWR023" H 850 4650 30  0001 C CNN
-F 1 "GND" H 850 4580 30  0001 C CNN
-F 2 "" H 850 4650 60  0000 C CNN
-F 3 "" H 850 4650 60  0000 C CNN
-	1    850  4650
-	0    1    1    0
+P 1250 4350
+F 0 "#PWR023" H 1250 4350 30  0001 C CNN
+F 1 "GND" H 1250 4280 30  0001 C CNN
+F 2 "" H 1250 4350 60  0000 C CNN
+F 3 "" H 1250 4350 60  0000 C CNN
+	1    1250 4350
+	-1   0    0    1
 $EndComp
 Wire Wire Line
@@
 Text Label 2200 2150 0    60   ~ 0
 VCC
-Text Label 1250 4350 0    60   ~ 0
+Text Label 850  4650 0    60   ~ 0
 VCC
 Text Label 2700 3450 2    60   ~ 0
@@
 Text Label 3175 8200 0    60   ~ 0
 SCL
+Text Label 1250 4850 2    60   ~ 0
+SDA
 Text Label 1250 4750 2    60   ~ 0
-SDA
-Text Label 1250 4850 2    60   ~ 0
 SCL
 Text Label 14975 5450 2    60   ~ 0
