File: watch-v4/watch-v4.sch (KiCad schematic (older format))
At the start: 44 parts, among them J1 CONN_10, P1 Expansion Header, Q1 MOSFET_P, Q2 BSS138, U1 IC_MCP73831, U2 MAX1722, U3 DS3231, U4 LSM9DS0, U5 NRF51822, U6 BALUN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

Commit message: v6 as sent to fab (errors!)
Parts:
- removed D3, D4, D5: LED, Capacitors_SMD:C_0603, symbol LED
- removed Q2: BSS138, TO_SOT_Packages_SMD:SOT-23, symbol BSS138
- removed R9: 47, Resistors_SMD:R_0603, symbol R_Small
Changed lines of the file:
@@
 Wire Wire Line
 	6075 2750 6075 2950
-$Comp
-L GND #PWR022
-U 1 1 570C1180
-P 15425 8100
-F 0 "#PWR022" H 15425 7850 50  0001 C CNN
-F 1 "GND" H 15425 7950 50  0000 C CNN
-F 2 "" H 15425 8100 60  0000 C CNN
-F 3 "" H 15425 8100 60  0000 C CNN
-	1    15425 8100
-	1    0    0    -1
-$EndComp
 Text Label 4350 2200 0    60   ~ 0
-Backlight
-Text Label 14575 7875 0    60   ~ 0
 Backlight
 Text Label 4350 4850 0    60   ~ 0
@@
 	1250 4350 1250 4550
 $Comp
-L GND-RESCUE-watch-v4 #PWR023
+L GND-RESCUE-watch-v4 #PWR022
 U 1 1 58005D02
 P 1250 4350
-F 0 "#PWR023" H 1250 4350 30  0001 C CNN
+F 0 "#PWR022" H 1250 4350 30  0001 C CNN
 F 1 "GND" H 1250 4280 30  0001 C CNN
 F 2 "" H 1250 4350 60  0000 C CNN
@@
 	4350 2650 4650 2650
 $Comp
-L GND #PWR024
+L GND #PWR023
 U 1 1 5800C121
 P 4850 2650
-F 0 "#PWR024" H 4850 2400 50  0001 C CNN
+F 0 "#PWR023" H 4850 2400 50  0001 C CNN
 F 1 "GND" H 4850 2500 50  0000 C CNN
 F 2 "" H 4850 2650 60  0000 C CNN
@@
 $EndComp
 $Comp
-L GND #PWR025
+L GND #PWR024
 U 1 1 5800C273
 P 4550 4000
-F 0 "#PWR025" H 4550 3750 50  0001 C CNN
+F 0 "#PWR024" H 4550 3750 50  0001 C CNN
 F 1 "GND" H 4550 3850 50  0000 C CNN
 F 2 "" H 4550 4000 60  0000 C CNN
@@
 	11025 2550 11025 2800
 $Comp
-L GND #PWR026
+L GND #PWR025
 U 1 1 5800CB9B
 P 11025 3100
-F 0 "#PWR026" H 11025 2850 50  0001 C CNN
+F 0 "#PWR025" H 11025 2850 50  0001 C CNN
 F 1 "GND" H 11025 2950 50  0000 C CNN
 F 2 "" H 11025 3100 60  0000 C CNN
@@
 	1275 8250 1725 8250
 Connection ~ 1525 8250
-$Comp
-L LED D5
-U 1 1 5801039E
-P 15225 7425
-F 0 "D5" H 15225 7525 50  0000 C CNN
-F 1 "LED" H 15225 7325 50  0000 C CNN
-F 2 "Capacitors_SMD:C_0603" H 15325 7225 60  0001 C CNN
-F 3 "~" H 15225 7425 60  0000 C CNN
-	1    15225 7425
-	-1   0    0    1
-$EndComp
-$Comp
-L LED D4
-U 1 1 58010482
-P 15225 7100
-F 0 "D4" H 15225 7200 50  0000 C CNN
-F 1 "LED" H 15225 7000 50  0000 C CNN
-F 2 "Capacitors_SMD:C_0603" H 15325 6900 60  0001 C CNN
-F 3 "~" H 15225 7100 60  0000 C CNN
-	1    15225 7100
-	-1   0    0    1
-$EndComp
-$Comp
-L LED D3
-U 1 1 58010529
-P 15225 6775
-F 0 "D3" H 15225 6875 50  0000 C CNN
-F 1 "LED" H 15225 6675 50  0000 C CNN
-F 2 "Capacitors_SMD:C_0603" H 15325 6575 60  0001 C CNN
-F 3 "~" H 15225 6775 60  0000 C CNN
-	1    15225 6775
-	-1   0    0    1
-$EndComp
-$Comp
-L BSS138 Q2
-U 1 1 58010CCE
-P 15325 7825
-F 0 "Q2" H 15525 7900 50  0000 L CNN
-F 1 "BSS138" H 15525 7825 50  0000 L CNN
-F 2 "TO_SOT_Packages_SMD:SOT-23" H 15525 7750 50  0000 L CIN
-F 3 "" H 15325 7825 50  0000 L CNN
-	1    15325 7825
-	1    0    0    -1
-$EndComp
-Wire Wire Line
-	15425 8025 15425 8100
-Wire Wire Line
-	15125 7875 14575 7875
-$Comp
-L R_Small R9
-U 1 1 58011E7A
-P 14750 6775
-F 0 "R9" H 14780 6795 50  0000 L CNN
-F 1 "47" H 14780 6735 50  0000 L CNN
-F 2 "Resistors_SMD:R_0603" H 14750 6775 50  0001 C CNN
-F 3 "" H 14750 6775 50  0000 C CNN
-	1    14750 6775
-	0    -1   -1   0
-$EndComp
-Wire Wire Line
-	14500 6775 14650 6775
-Wire Wire Line
-	14850 6775 15025 6775
-Wire Wire Line
-	15025 6775 15025 7425
-Connection ~ 15025 7100
-Wire Wire Line
-	15425 6775 15425 7625
-Connection ~ 15425 7100
-Connection ~ 15425 7425
 Text Label 15675 4025 0    60   ~ 0
 VCC
 Text Label 14775 5850 2    60   ~ 0
 VCC
-Text Label 14500 6775 2    60   ~ 0
-VCC
 Text Label 5775 7525 2    60   ~ 0
